File: Incubator_Quetta-Client.kicad_sch (KiCad schematic)
At the start: 39 parts, among them J1 I2C_LCD, J10 3.3V CON, J11 Barrel_Jack_Switch_Pin3Ring, J12 MOTOR, J13 ALT_HEATER, J14 LIMIT SWITCHES, J15 DHT22, J2 AH20 (I2C), J3 LIVE_CON, J4 Fan, J5 Humidifier, J6 HEATER, J7 12V CON, J8 Rotary encoder, J9 5V CON, K1 MOTOR_RELAY, K2 HEATER_RELAY, Q1 BC547, Q2 BC547, Q3 IRF540N, Q4 IRF540N, U1 DEVKIT_V1_ESP32-WROOM-32, U2 BOB-12009, U3 LM7805_TO220, U4 LM1117DT-3.3

Commit message: basic layout done
Parts:
- added C3: 100uF, Capacitor_THT:C_Radial_D6.3mm_H5.0mm_P2.50mm, symbol Device:C
- J1: renamed from J4; footprint (none) -> Connector_PinHeader_2.54mm:PinHeader_1x02_P2.54mm_Horizontal
- J10: renamed from J8; footprint (none) -> Connector_PinHeader_2.54mm:PinHeader_1x05_P2.54mm_Vertical
- J11: renamed from J1; footprint (none) -> Connector_PinHeader_2.54mm:PinHeader_1x04_P2.54mm_Vertical
- J12: renamed from J2; footprint (none) -> Connector_PinHeader_2.54mm:PinHeader_1x04_P2.54mm_Vertical
- J13: renamed from J3; footprint (none) -> TerminalBlock_Altech:Altech_AK100_1x02_P5.00mm
- J2: renamed from J5; footprint (none) -> Connector_PinHeader_2.54mm:PinHeader_1x02_P2.54mm_Horizontal
- J4: renamed from J7; footprint (none) -> Connector_PinHeader_2.54mm:PinHeader_1x02_P2.54mm_Vertical
- J5: renamed from J9; footprint (none) -> Connector_PinHeader_2.54mm:PinHeader_1x02_P2.54mm_Vertical
- J6: renamed from J10; footprint (none) -> Connector_PinHeader_2.54mm:PinHeader_1x02_P2.54mm_Vertical
- J7: renamed from J13; footprint (none) -> Connector_PinHeader_2.54mm:PinHeader_1x02_P2.54mm_Vertical
- J8: renamed from J15; footprint (none) -> Connector_PinHeader_2.54mm:PinHeader_1x03_P2.54mm_Vertical
- J9: renamed from J14; footprint (none) -> Connector_PinHeader_2.54mm:PinHeader_1x04_P2.54mm_Vertical
- R1: renamed from R5; value 120 -> 330; footprint (none) -> Resistor_THT:R_Axial_DIN0204_L3.6mm_D1.6mm_P5.08mm_Horizontal
- R2: renamed from R4; value 330 -> 10k; footprint (none) -> Connector_PinHeader_2.54mm:PinHeader_1x04_P2.54mm_Vertical
- R3: renamed from R6; value 120 -> 330; footprint (none) -> Connector_PinHeader_2.54mm:PinHeader_1x04_P2.54mm_Vertical
- R4: renamed from R3; value 330 -> 10k; footprint (none) -> Connector_PinHeader_2.54mm:PinHeader_1x04_P2.54mm_Vertical
- R5: renamed from R2; footprint (none) -> Connector_PinHeader_2.54mm:PinHeader_1x04_P2.54mm_Vertical
- U4: renamed from U1; footprint DEVKIT_V1_ESP32-WROOM-32:MODULE_DEVKIT_V1_ESP32-WROOM-32 -> wroom_esp32_module:MODULE_ESP32_DEVKIT_V1
- renumbered C3 to C4, C4 to C5, D3 to D1, D1 to D2, D2 to D3, J12 to J14, J6 to J15, J11 to J3, Q4 to Q1, Q3 to Q2, Q1 to Q3, Q2 to Q4, R1 to R6, U3 to U1, U4 to U2, U2 to U3
Connections:
- net +12V: now also C3.1
- net DHT22: now also U4.28 (IO17)
- net GND: now also U4.14 (GND1), U4.32 (GND2), C3.2
- net LIM1: now also U4.7 (IO32)
- net LIM2: now also U4.8 (IO33)
- no-connect marks 4 -> 28
Other:
- note added: "2.9V"
- note removed: "***check capacitor values"
- note removed: "CHECK WHAT RESISTORS YOU NEED FOR THIS"

Commit message: finalised pcb. all done. waiting for approval
Parts:
- removed F1: Fuse, Fuse:Fuseholder_Cylinder-5x20mm_Schurter_OGN-SMD_Horizontal_Open, symbol Device:Fuse
- removed J3: Barrel_Jack_Switch_Pin3Ring, Connector_BarrelJack:BarrelJack_GCT_DCJ200-10-A_Horizontal, symbol Connector:Barrel_Jack_Switch_Pin3Ring
- added J16: 12V_CON, TerminalBlock_Altech:Altech_AK100_1x02_P5.00mm, symbol Connector:Screw_Terminal_01x02
Connections:
- net +12V: now also C3.2, J16.1 (Pin_1); no longer C3.1
- net AC_L: now also J14.2 (Pin_2); no longer J14.1 (Pin_1), K1.3, K2.3
- net GND: now also C3.1, J16.2 (Pin_2); no longer C3.2
- net M2: now also J14.1 (Pin_1); no longer J14.2 (Pin_2)
- net FUSE-CON renamed AC_N
- net AC_N: now also K1.3, K2.3
Other:
- moved on the sheet: C3
