File: Incubator_Quetta-Client.kicad_pcb (KiCad board)
At the start: 2 copper layers, 40 parts, among them J1 Fan, J10 Rotary encoder, J11 I2C_LCD, J12 AH20 (I2C), J13 LIVE_CON, J14 MOTOR, J15 HEATER, J2 Humidifier, J3 Barrel_Jack_Switch_Pin3Ring, J4 12V CON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

Commit message: finalised pcb. all done. waiting for approval
Parts:
- removed F1: Fuse, Fuse:Fuseholder_Cylinder-5x20mm_Schurter_OGN-SMD_Horizontal_Open
- removed J3: Barrel_Jack_Switch_Pin3Ring, Connector_BarrelJack:BarrelJack_Horizontal
- added G***: LOGO, logo:Capistor_logo, F.Cu at (155.3, 89.4)
- added J16: 12V_CON, TerminalBlock_Altech:Altech_AK100_1x02_P5.00mm, F.Cu at (113.9, 101.7)
- added REF**: MountingHole_2.2mm_M2, MountingHole:MountingHole_2.2mm_M2, F.Cu at (111.8, 53.8)
- added REF**: MountingHole_2.2mm_M2, MountingHole:MountingHole_2.2mm_M2, F.Cu at (111.3, 137.2)
- added REF**: MountingHole_2.2mm_M2, MountingHole:MountingHole_2.2mm_M2, F.Cu at (186.7, 137.7)
- added REF**: MountingHole_2.2mm_M2, MountingHole:MountingHole_2.2mm_M2, F.Cu at (188.2, 53.8)
- Q3, Q4: footprint Package_TO_SOT_THT:TO-92_Inline -> Package_TO_SOT_THT:TO-92_Inline_Wide
- U1: value LM7805_TO220 -> LM7805
- U4: footprint wroom_esp32_module:MODULE_ESP32_DEVKIT_V1 -> DEVKIT_V1_ESP32-WROOM-32:MODULE_DEVKIT_V1_ESP32-WROOM-32
- moved D2 100.6 mm to (132.8, 95.0)
- moved Q3 100.2 mm to (136.4, 100.1)
- moved J13 99.6 mm to (117.6, 62.0)
- moved R2 97.3 mm to (144.3, 118.6), turned to 180 degrees
- moved J14 96.9 mm to (131.7, 62.0)
- moved R4 91.8 mm to (144.3, 122.4), turned to 180 degrees
- moved J15 90.0 mm to (145.3, 62.2)
- moved Q4 89.0 mm to (144.8, 100.1)
- moved D3 86.6 mm to (137.4, 94.5), turned to 0 degrees
- moved K2 82.4 mm to (140.6, 88.5)
- moved K1 82.0 mm to (119.1, 88.5)
- moved R6 81.1 mm to (139.2, 104.1)
- moved J10 80.9 mm to (181.1, 120.1)
- moved J9 79.5 mm to (158.3, 115.6), turned to 90 degrees
- moved R5 77.1 mm to (144.3, 107.7), turned to 180 degrees
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Connections:
- C3 pad 1: +12V -> GND
- C3 pad 2: GND -> +12V
- J13 pad 1: /FUSE-CON -> AC_N
- J14 pad 1: AC_L -> M2
- J14 pad 2: M2 -> AC_L
- K1 pad 3: AC_L -> AC_N
- K2 pad 3: AC_L -> AC_N
Routing:
- net GND: track 0.00 -> 178.6 mm, vias 0 -> 9
- net +5V: track 0.00 -> 170.3 mm, vias 0 -> 4
- net +3.3V: track 0.00 -> 158.9 mm, vias 0 -> 4
- net +12V: track 0.00 -> 79.5 mm
- net M2: track 0.00 -> 77.0 mm
- net HEATER_PIN: track 0.00 -> 70.4 mm
- net SDA_MCU: track 0.00 -> 68.2 mm
- net SCL_MCU: track 0.00 -> 66.2 mm
- net SCL: track 0.00 -> 49.9 mm, vias 0 -> 1
- net SDA: track 0.00 -> 47.6 mm
- net LIM2: track 0.00 -> 45.9 mm, vias 0 -> 2
- net DHT22: track 0.00 -> 45.3 mm, vias 0 -> 1
- net LIM1: track 0.00 -> 43.7 mm, vias 0 -> 2
- net HEATER-: track 0.00 -> 41.7 mm
- net ROT_DATA: track 0.00 -> 40.5 mm
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- added copper zone on F.Cu, net +12V
- added copper zone on F.Cu, net AC_L
- added copper zone on F.Cu, net AC_N
- added copper zone on F.Cu, net GND
- added copper zone on F.Cu, net HEATER-
- added copper zone on F.Cu, net M2
Other:
- board outline added: 83.7 x 90.3 mm
- board text added: "V1.3"

Commit message: final
Parts:
- removed G***: LOGO, logo:Capistor_logo
- moved C1 0.19 mm to (111.4, 113.0)
Routing:
- net +3.3V: track 158.9 -> 156.3 mm
- net SCL_MCU: track 66.2 -> 68.5 mm
- net SCL: track 49.9 -> 50.8 mm
- net +12V: track 79.5 -> 80.4 mm
- net Net-(Q2-G): track 18.0 -> 18.7 mm
- net HUMIDIFIER_PIN: track 39.0 -> 39.6 mm
